Commit message: Added plugin for collision counter

File: zuuu_description/urdf/zuuu.gazebo.xacro (robot description, xacro)
@@ -36,4 +36,19 @@
             </plugin>
         </gazebo>
+        <gazebo reference="base_link">
+            <sensor name="base_contact_sensor" type="contact">
+                <always_on>true</always_on>
+                <update_rate>50</update_rate>
+                <contact>
+                    <collision>base_link_collision</collision>
+                </contact>
+                <plugin name="gazebo_ros_bumper" filename="libgazebo_ros_bumper.so">
+                    <ros>
+                        <remapping>bumper_states:=/reachy/contacts_state</remapping>
+                    </ros>
+                    <frame_name>base_link</frame_name>
+                </plugin>
+            </sensor>
+        </gazebo>
         <gazebo reference="lidar_link">
             <sensor name="lidar" type="ray">
